File: hardware/color.kicad_pcb (KiCad board)
At the start: 2 copper layers, 25 x 20 mm, 20 parts, among them P1 CON-SENSOR, Q1 2N7002P, U1 TCS3472, U2 M24C64, U3 DRILL, U4 DRILL, U5 DRILL, U6 DRILL

Commit message: Add 3d information (final)
Parts:
- C1, C2: footprint 0603 -> kicad-libraries:C0603
- D1: footprint LED-3x2 -> kicad-libraries:LED-3x2
- Fiducial_Mark (x2): footprint Fiducial_Mark -> kicad-libraries:Fiducial_Mark
- G***: footprint Logo_31x31 -> kicad-libraries:Logo_31x31
- P1: footprint CON-SENSOR -> kicad-libraries:CON-SENSOR
- Q1: footprint SOT23GDS -> kicad-libraries:SOT23GDS
- R1, R2, R3, R4: footprint 0603 -> kicad-libraries:R0603
- U1: footprint FN-TCS3472 -> kicad-libraries:FN-TCS3472
- U2: footprint SOIC8 -> kicad-libraries:SOIC8
- U3, U4, U5, U6: footprint DRILL_NP -> kicad-libraries:DRILL_NP
- VAL: footprint WEEE_7mm -> kicad-libraries:WEEE_7mm
- VAL: footprint CE_5mm -> kicad-libraries:CE_5mm
- turned VAL to 180 degrees
Connections:
- P1 pad 1: (no net) -> Net-(P1-Pad1)
- U1 pad 4: (no net) -> Net-(U1-Pad4)
- U2 pad 7: (no net) -> Net-(U2-Pad7)
